File: adapter_pcb_v2/adapter_pcb.kicad_pcb (KiCad board)
At the start: 2 copper layers, 39.9 x 39.9 mm, 12 parts, among them J1 Conn_01x04, J2 Conn_01x02, J3 Screw_Terminal_01x02, J4 Conn_01x02, SW1 SW_SPST, U1 74AHC1G14

Commit message: Add silkscreen for ordering
Parts:
- added G***: LOGO, LOGO, F.Cu at (127.7, 75.2)
Other:
- board text added: "FRoDO Main Release"
- board text added: "JLCJLCJLCJLC"
- board text added: "rev 1"
